Commit message: intermediate commit

File: rotors_description/urdf/crazyflie2_forster.xacro (robot description, xacro)
@@ -22,5 +22,6 @@
   <xacro:property name="use_mesh_file" value="true" />
   <xacro:property name="mesh_file" value="package://rotors_description/meshes/crazyflie2.dae" />
-  <xacro:property name="mass" value="0.025" /> <!-- [kg] -->
+  <!--xacro:property name="mass" value="0.025" /--> <!-- [kg] -->
+  <xacro:property name="mass" value="0.031" /> <!-- [kg], with passive marker board -->
   <xacro:property name="body_width" value="0.045" /> <!-- [m] -->
   <xacro:property name="body_height" value="0.03" /> <!-- [m] -->
