Commit message: use forster params

File: rotors_description/urdf/crazyflie2_base.xacro (robot description, xacro)
@@ -19,5 +19,5 @@
   <xacro:include filename="$(find rotors_description)/urdf/component_snippets.xacro" />
   <!-- Instantiate crazyflie2 "mechanics" -->
-  <xacro:include filename="$(find rotors_description)/urdf/crazyflie2.xacro" />
+  <xacro:include filename="$(find rotors_description)/urdf/crazyflie2_forster.xacro" />
   <!-- Instantiate a controller.  -->
   <xacro:controller_plugin_macro namespace="${namespace}" imu_sub_topic="imu" />

File: rotors_description/urdf/crazyflie2_forster.xacro (robot description, xacro)
@@ -22,5 +22,6 @@
   <xacro:property name="use_mesh_file" value="true" />
   <xacro:property name="mesh_file" value="package://rotors_description/meshes/crazyflie2.dae" />
-  <xacro:property name="mass" value="0.025" /> <!-- [kg] -->
+  <!--xacro:property name="mass" value="0.025" /--> <!-- [kg] -->
+  <xacro:property name="mass" value="0.031" /> <!-- [kg], with passive marker board -->
   <xacro:property name="body_width" value="0.045" /> <!-- [m] -->
   <xacro:property name="body_height" value="0.03" /> <!-- [m] -->
